Commit message: refactor + simple devop

File: mybot/robot.urdf (robot description, URDF)
Before this commit: robot mybot, 7 links, 6 joints
Links:
- link arm1: mass 1.26286 -> 0.074836
- link arm1_2: mass 1.26286 -> 0.074836
- link arm2: mass 0.575994 -> 0.0341329
- link arm2_2: mass 0.575994 -> 0.0341329
- link base: mass 6.33654 -> 0.375499
- link hand: mass 0.11732 -> 0.00695227
- link swivle: mass 1.06472 -> 0.0630945
Joints:
- joint base_rot: origin xyz=-0.0595984 0.133273 0.0574778 rpy=3.14159 -0 2.48016 -> xyz=-0.0595984 0.133273 0.0574778 rpy=3.14159 -0 -2.95606
- joint joint1: origin xyz=-0.0127 -0 -0.0762 rpy=1.5708 -0.800967 -1.5708 -> xyz=-0.0127 0 -0.0762 rpy=1.5708 -0.550725 -1.5708
- joint joint2: origin xyz=-0.120251 -0.0936238 -0 rpy=-0 0 -1.26071 -> xyz=-0.120251 -0.0936238 -0 rpy=0 0 1.71304
- joint joint4: origin xyz=0.0112995 -0.00579758 -0.2032 rpy=1.5708 -1.48999 1.09674 -> xyz=-0.0122913 0.00319579 -0.2032 rpy=1.5708 1.08193 -1.82517
- joint wrist5: origin xyz=-0.146016 -0.101451 -0.0127 rpy=-1.5708 -1.20722 -0.963574 -> xyz=-0.146016 -0.101451 -0.0127 rpy=1.5708 -0.103846 2.17802
